File: hardware/usb-sniffer.kicad_pcb (KiCad board)
At the start: 2 copper layers, 58.2 x 38.1 mm, 87 parts, among them IC1 LCMXO2-2000HC, IC10 DSC6101CI2A-024.0000, IC2 MIC5504-3.3v, IC3 MAX9032AKA+T, IC4 USB3343, IC5 MAX9032AKA+T, IC6 DSC6101CI2A-026.0000, IC7 MAX9032AKA+T, IC8 I2C-EEPROM, IC9 CY7C68013A-56PVXC, J1 USB-C, J2 USB-C, J3 USB-A, J4 IN, J5 GND

Commit message: Added EEPROM part name
Parts:
- IC1: value LCMXO2-2000HC -> LCMXO2-2000HC-5TG100
- IC8: value I2C-EEPROM -> 24LC128
Changed lines of the file:
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@@
         (effects (font (size 1 1) (thickness 0.127)))
     )
-    (fp_text value "I2C-EEPROM" (at 0 0) (layer "F.Fab")
+    (fp_text value "24LC128" (at 0 0) (layer "F.Fab")
         (effects (font (size 0.7 0.7) (thickness 0.1)))
     )
@@
         (effects (font (size 1 1) (thickness 0.127)))
     )
-    (fp_text value "LCMXO2-2000HC" (at 0 0) (layer "F.Fab")
+    (fp_text value "LCMXO2-2000HC-5TG100" (at 0 0) (layer "F.Fab")
         (effects (font (size 0.5 0.5) (thickness 0.1)))
     )

Commit message: Fixed resistor value
Parts:
- R6: value 512 -> 510
Changed lines of the file:
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@@
         (effects (font (size 1 1) (thickness 0.127)))
     )
-    (fp_text value "512" (at 0 -0.016 180 unlocked) (layer "F.Fab")
+    (fp_text value "510" (at 0 -0.016 180 unlocked) (layer "F.Fab")
         (effects (font (size 0.5 0.5) (thickness 0.05)))
     )
